File: Docs/A500-EXT-IDE.v1.0.0.sch (EAGLE design)
At the start: 47 parts, among them CN1 A500-EXPANSION-SLOT-SOLDER, IC10 50MHz, IC2 XC95288XL-TQ144, IC3 74HCT245PW, IC4 74HCT245PW, IC5 74HCT245PW, IC6 AS4C4M16S-6TCN, IC7 LD117AS33TR, IC8 AM29F010J-SOCKET

Commit message: Add files via upload
Connections:
- new net !C1: CN1.!CCK!, IC2.P$93-FB16MC05
- new net !C3: CN1.!CCKQ!, IC2.P$94-FB16MC06
- new net CDAC: CN1.CDAC, IC2.P$92-FB16MC03
Changed lines of the file:
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@@
+</segment>
+</net>
+<net name="CDAC" class="0">
+<segment>
+<pinref part="CN1" gate="G$1" pin="CDAC"/>
+<wire x1="43.18" y1="129.54" x2="25.4" y2="129.54" width="0.1524" layer="91"/>
+<label x="25.4" y="129.54" size="1.778" layer="95"/>
+</segment>
+</net>
+<net name="!C3" class="0">
+<segment>
+<pinref part="CN1" gate="G$1" pin="!CCKQ!"/>
+<wire x1="74.93" y1="132.08" x2="86.36" y2="132.08" width="0.1524" layer="91"/>
+<label x="83.82" y="132.08" size="1.778" layer="95"/>
+</segment>
+</net>
+<net name="!C1" class="0">
+<segment>
+<pinref part="CN1" gate="G$1" pin="!CCK!"/>
+<wire x1="74.93" y1="129.54" x2="86.36" y2="129.54" width="0.1524" layer="91"/>
+<label x="83.82" y="129.54" size="1.778" layer="95"/>
 </segment>
 </net>
@@
 </segment>
 </net>
+<net name="CDAC" class="0">
+<segment>
+<pinref part="IC2" gate="G$1" pin="P$92-FB16MC03"/>
+<wire x1="144.78" y1="91.44" x2="149.86" y2="91.44" width="0.1524" layer="91"/>
+<label x="149.86" y="91.44" size="1.778" layer="95"/>
+</segment>
+</net>
+<net name="!C1" class="0">
+<segment>
+<pinref part="IC2" gate="G$1" pin="P$93-FB16MC05"/>
+<wire x1="144.78" y1="93.98" x2="149.86" y2="93.98" width="0.1524" layer="91"/>
+<label x="149.86" y="93.98" size="1.778" layer="95"/>
+</segment>
+</net>
+<net name="!C3" class="0">
+<segment>
+<pinref part="IC2" gate="G$1" pin="P$94-FB16MC06"/>
+<wire x1="144.78" y1="96.52" x2="149.86" y2="96.52" width="0.1524" layer="91"/>
+<label x="149.86" y="96.52" size="1.778" layer="95"/>
+</segment>
+</net>
